File: usb.kicad_sch (KiCad schematic)
At the start: 4 parts, among them J9 USB_C_Receptacle_USB2.0_16P

Commit message: Committing project.
Parts:
- J9: footprint (none) -> noaidi-fpga-synth:GCT_USB4085-GF-A_REVB
Connections:
- net at FB2.1: now also J9.S1 (SHIELD), J9.S2 (SHIELD), J9.S3 (SHIELD), J9.S4 (SHIELD); no longer J9.SH (SHIELD)
Changed lines of the file:
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@@
+	(wire
+		(pts
+			(xy 146.05 101.6) (xy 148.59 101.6)
+		)
+		(stroke
+			(width 0)
+			(type default)
+		)
+	)
+	(wire
+		(pts
+			(xy 146.05 88.9) (xy 157.48 88.9)
+		)
+		(stroke
+			(width 0)
+			(type default)
+		)
+	)
+	(wire
+		(pts
+			(xy 130.81 119.38) (xy 130.81 130.81)
+		)
+		(stroke
+			(width 0)
+			(type default)
+		)
+	)
 	(wire
 		(pts
 			(xy 123.19 127) (xy 123.19 130.81)
-		)
-		(stroke
-			(width 0)
-			(type default)
-		)
-	)
-	(wire
-		(pts
-			(xy 146.05 101.6) (xy 148.59 101.6)
-		)
-		(stroke
-			(width 0)
-			(type default)
-		)
-	)
-	(wire
-		(pts
-			(xy 146.05 88.9) (xy 157.48 88.9)
-		)
-		(stroke
-			(width 0)
-			(type default)
-		)
-	)
-	(wire
-		(pts
-			(xy 130.81 119.38) (xy 130.81 130.81)
 		)
 		(stroke
@@
 			)
 		)
-		(property "Footprint" ""
+		(property "Footprint" "noaidi-fpga-synth:GCT_USB4085-GF-A_REVB"
 			(at 134.62 96.52 0)
 			(hide yes)
@@
 		(pin "B5"
 		)
-		(pin "SH"
+		(pin "S4"
 		)
 		(pin "B6"
@@
 		(pin "B1"
 		)
+		(pin "S2"
+		)
+		(pin "S3"
+		)
+		(pin "S1"
+		)
 		(instances
